File: lin_hw.kicad_sch (KiCad schematic)
At the start: 53 parts, among them J1 USB_C_Receptacle_USB2.0_16P, J6 Conn_01x10, J8 Barrel_Jack_MountingPin, U1 FT4232H, U3 AP2112K-3.3, U4 93CxxB, U8 74HC595, Y1 12Mhz

Commit message: routed
Parts:
- removed D10, D11, D12, D9: LED, ftdi_quad_lin:fix_lem_180, symbol Device:LED
- added D10, D9: ~, ftdi_quad_lin:1296.3004, symbol ftdi_quad_lin:led_array_4
- added R22, R23, R24, R25: 2.4k, Resistor_SMD:R_0805_2012Metric, symbol Device:R
- J6: footprint Connector_PinHeader_2.54mm:PinHeader_1x10_P2.54mm_Vertical -> Connector_PinHeader_2.54mm:PinHeader_1x11_P2.54mm_Vertical; symbol Connector_Generic:Conn_01x10 -> Connector_Generic:Conn_01x11
Connections:
- net +3V3: now also J6.9 (Pin_9)
- net +5V: now also J6.10 (Pin_10); no longer J6.1 (Pin_1)
- net GND: now also J6.11 (Pin_11), D10.1, D10.3, D10.5, D10.7, D9.1, D9.3, D9.5, D9.7; no longer J6.10 (Pin_10)
- net LIN0_RXD: now also J6.2 (Pin_2); no longer J6.3 (Pin_3)
- net LIN0_TXD: now also J6.1 (Pin_1); no longer J6.2 (Pin_2)
- net LIN1_RXD: now also J6.4 (Pin_4); no longer J6.5 (Pin_5)
- net LIN1_TXD: now also J6.3 (Pin_3); no longer J6.4 (Pin_4)
- net LIN2_RXD: now also J6.6 (Pin_6); no longer J6.7 (Pin_7)
- net LIN2_TXD: now also J6.5 (Pin_5); no longer J6.6 (Pin_6)
- net LIN3_RXD: now also J6.8 (Pin_8); no longer J6.9 (Pin_9)
- net LIN3_TXD: now also J6.7 (Pin_7); no longer J6.8 (Pin_8)
- net at R19.1: now also D9.4
- net at R21.1: now also D9.8
- net at R20.1: now also D9.6
- net at R17.1: now also D9.2
- new net: D10.4, R23.1
- new net: D10.2, R22.1
- new net: D10.6, R24.1
- new net: D10.8, R25.1
- new net LIN 0/VBAT: R22.2
- new net LIN 1/VBAT: R23.2
- new net LIN 2/VBAT: R24.2
- new net LIN 3/VBAT: R25.2
Other:
- sheet LIN 0 ports: added VBAT; removed none
- sheet LIN 1 ports: added VBAT; removed none
- sheet LIN 2 ports: added VBAT; removed none
- sheet LIN 3 ports: added VBAT; removed none
