File: lin_hw.kicad_pcb (KiCad board)
At the start: 2 copper layers, 70.8 x 53 mm, 93 parts, among them J1 USB_C_Receptacle_USB2.0_16P, J2 Screw_Terminal_01x03, J3 Screw_Terminal_01x03, J4 Screw_Terminal_01x03, J5 Screw_Terminal_01x03, J6 Conn_01x10, J8 Barrel_Jack_MountingPin, U1 FT4232H, U2 TJA1029T, U3 AP2112K-3.3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

Commit message: routed
Parts:
- removed D11, D12: LED, ftdi_quad_lin:fix_lem_180
- added R22: 2.4k, Resistor_SMD:R_0805_2012Metric, F.Cu at (113.1, 82.0)
- added R23: 2.4k, Resistor_SMD:R_0805_2012Metric, F.Cu at (113.1, 79.5)
- added R24: 2.4k, Resistor_SMD:R_0805_2012Metric, F.Cu at (113.1, 77.0)
- added R25: 2.4k, Resistor_SMD:R_0805_2012Metric, F.Cu at (113.1, 74.2)
- D10, D9: value LED -> ~; footprint ftdi_quad_lin:fix_lem_180 -> ftdi_quad_lin:1296.3004
- J6: footprint Connector_PinHeader_2.54mm:PinHeader_1x10_P2.54mm_Vertical -> Connector_PinHeader_2.54mm:PinHeader_1x11_P2.54mm_Vertical
- moved D9 34.8 mm to (101.8, 78.2), turned to 90 degrees
- moved U3 33.2 mm to (91.8, 119.0)
- moved R17 32.3 mm to (96.8, 82.0), turned to 180 degrees
- moved C16 29.4 mm to (95.4, 119.0), turned to -90 degrees
- moved R20 27.2 mm to (96.8, 76.7), turned to 180 degrees
- moved C15 26.8 mm to (90.2, 116.0), turned to 0 degrees
- moved R19 25.5 mm to (96.9, 79.5), turned to 180 degrees
- moved FB3 24.6 mm to (94.2, 116.2), turned to 180 degrees
- moved R4 23.6 mm to (90.8, 105.0), turned to 90 degrees
- moved D10 22.8 mm to (108.3, 78.2), turned to 90 degrees
- moved R5 19.6 mm to (90.8, 110.8), turned to -90 degrees
- moved C2 19.4 mm to (93.0, 111.5), turned to -90 degrees
- moved J1 17.9 mm to (84.9, 109.4)
- moved J8 17.1 mm to (93.5, 85.5)
- moved H3 17.0 mm to (84.8, 118.2)
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Connections:
- net Net-(D1-A) renamed /LIN 0/VBAT
- net Net-(D3-A) renamed /LIN 1/VBAT
- net Net-(D5-A) renamed /LIN 2/VBAT
- net Net-(D7-A) renamed /LIN 3/VBAT
- D10 pad 2: Net-(D10-A) -> Net-(D10-Pad2)
- J6 pad 1: +5V -> /LIN0_TXD
- J6 pad 10: GND -> +5V
- J6 pad 2: /LIN0_TXD -> /LIN0_RXD
- J6 pad 3: /LIN0_RXD -> /LIN1_TXD
- J6 pad 4: /LIN1_TXD -> /LIN1_RXD
- J6 pad 5: /LIN1_RXD -> /LIN2_TXD
- J6 pad 6: /LIN2_TXD -> /LIN2_RXD
- J6 pad 7: /LIN2_RXD -> /LIN3_TXD
- J6 pad 8: /LIN3_TXD -> /LIN3_RXD
- J6 pad 9: /LIN3_RXD -> +3V3
- R19 pad 1: Net-(D10-A) -> Net-(D9-Pad4)
- R20 pad 1: Net-(D11-A) -> Net-(D9-Pad6)
- R21 pad 1: Net-(D12-A) -> Net-(D9-Pad8)
Routing:
- net +5V: track 54.1 -> 214.8 mm, vias 0 -> 2
- net GND: track 0.00 -> 137.8 mm, vias 0 -> 65
- net +3V3: track 9.61 -> 84.5 mm, vias 0 -> 4
- net /LIN3_RXD: track 2.18 -> 57.6 mm, vias 0 -> 2
- net /LIN3_TXD: track 0.00 -> 41.6 mm, vias 0 -> 2
- net /LIN 2/VBAT: track 42.6 -> 81.2 mm
- net /LIN2_RXD: track 2.18 -> 37.6 mm, vias 0 -> 2
- net Net-(U8-QH): track 0.00 -> 32.2 mm
- net /LIN1_RXD: track 2.18 -> 33.3 mm, vias 0 -> 2
- net /LIN2_TXD: track 0.00 -> 30.9 mm, vias 0 -> 3
- net Net-(U8-QB): track 0.00 -> 30.3 mm
- net Net-(U8-QD): track 0.00 -> 30.0 mm
- net +1V8: track 9.65 -> 39.6 mm
- net /LIN1_TXD: track 0.00 -> 29.9 mm, vias 0 -> 2
- net /LIN0_RXD: track 2.18 -> 31.5 mm, vias 0 -> 2
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- added copper zone on B.Cu, net GND
- added copper zone on F.Cu, net GND
Other:
- board size 70.8 x 53 mm -> 53.8 x 53 mm
- board text added: "3V3"
- board text added: "5V"
- board text added: "GND"
- board text added: "RX0"
- board text added: "RX1"
- board text added: "RX2"
- board text added: "RX3"
- board text added: "TX0"
- board text added: "TX1"
- board text added: "TX2"
- board text added: "TX3"

Commit message: finito
Parts:
- moved H1 0.50 mm to (132.0, 72.2)
- moved H4 0.50 mm to (132.0, 118.2)
Routing:
- net GND: track 137.8 -> 148.0 mm
- net +1V8: track 39.6 -> 38.9 mm
Other:
- board size 53.8 x 53 mm -> 54.2 x 53 mm
- board text added: "0"
- board text added: "1"
- board text added: "2"
- board text added: "3"
- board text added: "data"
- board text added: "power"
- board text removed: "LIN 1"
- board text removed: "otoceny spravne?"
