File: ftdi_quad_lin.kicad_pcb (KiCad board)
At the start: 2 copper layers, 55 x 80 mm, 145 parts, among them J1 USB_C_Receptacle_USB2.0_16P, J2 Screw_Terminal_01x03, J3 Screw_Terminal_01x03, J4 Screw_Terminal_01x03, J5 Screw_Terminal_01x03, J6 Conn_01x10, J8 Barrel_Jack_MountingPin, Q1 MMBT2222A, Q10 MMBT2222A, Q11 MMBT2222A, Q12 MMBT2222A, Q2 MMBT2222A, Q3 MMBT2222A, Q4 MMBT2222A, Q5 MMBT2222A, Q6 MMBT2222A, Q7 MMBT2222A, Q8 MMBT2222A, Q9 MMBT2222A, U1 FT4232H, U2 TJA1029T, U3 AP2112K-3.3, U4 93CxxB, U5 TJA1029T, U6 TJA1029T, U7 TJA1029T, U8 74HC595, Y1 12Mhz

Commit message: reworking
Parts:
- added J7: Conn_01x05, Connector_JST:JST_XH_B5B-XH-A_1x05_P2.50mm_Vertical, F.Cu at (104.5, 64.8)
- added REF**: TerminalBlock_Phoenix_MKDS-1,5-2-5.08_1x02_P5.08mm_Horizont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, TerminalBlock_Phoenix:TerminalBlock_Phoenix_MKDS-1,5-2-5.08_1x02_P5.08mm_Horizontal, F.Cu at (193.0, 85.8)
- moved C31 102.5 mm to (174.4, 110.5)
- moved D11 102.5 mm to (177.0, 113.5)
- moved Q1 102.5 mm to (177.3, 108.6)
- moved R22 102.5 mm to (180.8, 109.7)
- moved R23 102.5 mm to (180.8, 111.7)
- moved R24 102.5 mm to (180.8, 113.7)
- moved R25 102.5 mm to (180.8, 107.7)
- moved R27 102.5 mm to (177.3, 111.5)
- moved C30 102.5 mm to (187.7, 109.1)
- moved Q2 102.5 mm to (184.7, 109.3)
- moved Q3 102.5 mm to (184.7, 112.8)
- moved R26 102.5 mm to (187.7, 112.8)
- moved Q7 57.9 mm to (177.3, 88.4)
- moved R34 57.9 mm to (180.8, 89.5)
- moved R35 57.9 mm to (180.8, 91.5)
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Routing:
- net +5V: track 165.0 -> 124.5 mm, vias 2 -> 0
- net +1V8: track 38.9 -> 2.67 mm
- net GND: track 60.9 -> 28.0 mm
- net +3V3: track 68.8 -> 39.2 mm, vias 3 -> 2
- net /LIN3_TXD: track 17.9 -> 0.00 mm, vias 1 -> 0
- net /LIN2_RXD: track 14.7 -> 2.18 mm, vias 1 -> 0
- net /LIN2_TXD: track 12.2 -> 0.00 mm, vias 2 -> 0
- net /USB_D-: track 14.2 -> 2.84 mm
- net /USB_D+: track 13.1 -> 2.59 mm
- net /VBAT2: track 9.78 -> 0.00 mm
- net Net-(D3-A): track 8.54 -> 0.00 mm
- net /eeprom/EECLK: track 17.3 -> 8.89 mm
- net Net-(D5-A): track 8.09 -> 0.00 mm
- net /LIN0_TXD: track 7.40 -> 0.00 mm
- net /LIN1_TXD: track 6.04 -> 0.00 mm
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Other:
- board text added: "VBAT_EXT"

Commit message: yep crash
Parts:
- removed the REF** at (193.0, 85.8)
- moved R17 62.6 mm to (183.0, 107.8), turned to -90 degrees
- moved J7 35.8 mm to (68.8, 62.8)
- moved R19 31.7 mm to (99.2, 59.0)
- moved C30 9.18 mm to (196.8, 108.3)
- moved D11 9.18 mm to (186.2, 112.7)
- moved Q2 9.18 mm to (193.8, 108.5)
- moved Q3 9.18 mm to (193.8, 112.1)
- moved R22 9.18 mm to (190.0, 108.9)
- moved R23 9.18 mm to (190.0, 110.9)
- moved R24 9.18 mm to (190.0, 112.9)
- moved R25 9.18 mm to (190.0, 106.9)
- moved R26 9.18 mm to (196.8, 112.0)
- moved R27 9.18 mm to (186.5, 110.7)
- moved Q1 9.18 mm to (186.4, 107.9)
- moved C31 8.64 mm to (183.0, 111.7)
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
Commit message: before givinr resistors
Parts:
- C30, C31, C32, C33, C34, C35, C36, C37, D10, D11, D12, D13, Q1, Q10, Q11, Q12, Q2, Q3, Q4, Q5, Q6, Q7, Q8, Q9, R17, R19, R20, R21, R22, R23, R24, R25, R26, R27, R28, R29, R30, R31, R32, R33, R34, R35, R36, R37, R38, R39, R40, R41, R42, R43, R44, R45: moved to B.Cu
- moved R24 141.4 mm to (59.5, 58.5)
- moved D11 141.3 mm to (55.6, 58.7)
- moved Q3 140.8 mm to (63.3, 59.3)
- moved R26 140.7 mm to (66.3, 59.4), turned to 90 degrees
- moved C31 140.5 mm to (52.5, 59.7), turned to 90 degrees
- moved R23 139.9 mm to (59.5, 60.5)
- moved R27 139.8 mm to (56.0, 60.7)
- moved R22 138.5 mm to (59.5, 62.5)
- moved Q2 138.3 mm to (63.3, 62.9)
- moved C30 138.1 mm to (66.3, 63.1), turned to 90 degrees
- moved Q1 137.8 mm to (55.9, 63.5), turned to 90 degrees
- moved R17 137.8 mm to (52.5, 63.6), turned to 90 degrees
- moved R25 137.2 mm to (59.5, 64.5)
- moved R43 125.9 mm to (59.6, 88.7)
- moved Q10 125.3 mm to (56.0, 87.7), turned to 90 degrees
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Routing:
- net /LIN3_RXD: track 2.18 -> 103.6 mm
- net /LIN3_TXD: track 0.00 -> 89.2 mm, vias 0 -> 2
- net /LIN2_RXD: track 2.18 -> 74.3 mm, vias 0 -> 2
- net Net-(D1-A): track 0.00 -> 67.7 mm
- net /LIN0_TXD: track 0.00 -> 66.7 mm
- net /LIN2_TXD: track 0.00 -> 65.2 mm, vias 0 -> 2
- net Net-(D3-A): track 0.00 -> 55.9 mm
- net /LIN1_TXD: track 0.00 -> 53.3 mm, vias 0 -> 2
- net /LIN0_RXD: track 2.18 -> 51.7 mm, vias 0 -> 2
- net Net-(D5-A): track 0.00 -> 39.4 mm
- net /LIN1_RXD: track 2.18 -> 39.5 mm
- net Net-(D7-A): track 8.36 -> 44.3 mm
- net +5V: track 124.5 -> 93.1 mm
- net Net-(D12-K): track 22.3 -> 0.00 mm
- net +1V8: track 2.67 -> 22.9 mm
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Other:
- board text removed: "VBAT_EXT"
