File: ftdi_quad_lin.kicad_pcb (KiCad board)
At the start: 2 copper layers, 55 x 80 mm, 146 parts, among them J1 USB_C_Receptacle_USB2.0_16P, J2 Screw_Terminal_01x03, J3 Screw_Terminal_01x03, J4 Screw_Terminal_01x03, J5 Screw_Terminal_01x03, J6 Conn_01x10, J7 Conn_01x05, J8 Barrel_Jack_MountingPin, Q1 MMBT2222A, Q10 MMBT2222A, Q11 MMBT2222A, Q12 MMBT2222A, Q2 MMBT2222A, Q3 MMBT2222A, Q4 MMBT2222A, Q5 MMBT2222A, Q6 MMBT2222A, Q7 MMBT2222A, Q8 MMBT2222A, Q9 MMBT2222A, U1 FT4232H, U2 TJA1029T, U3 AP2112K-3.3, U4 93CxxB, U5 TJA1029T, U6 TJA1029T, U7 TJA1029T, U8 74HC595, Y1 12Mhz

Commit message: routing details
Parts:
- removed REF** (x4): DSUB-9_Female_Vertical_P2.77x2.84mm, Connector_Dsub:DSUB-9_Female_Vertical_P2.77x2.84mm
- C30, C31, C32, C33, C34, C35, C36, C37, D10, D11, D12, D13, Q1, Q10, Q11, Q12, Q2, Q3, Q4, Q5, Q6, Q7, Q8, Q9, R17, R19, R20, R22, R23, R24, R25, R26, R27, R28, R29, R30, R31, R32, R33, R34, R35, R36, R37, R38, R39, R40, R41, R42, R43, R44, R45: moved to F.Cu
- R21: value 330R -> 1k; moved to F.Cu
- moved R24 78.1 mm to (120.6, 107.2)
- moved D11 77.9 mm to (116.7, 107.0)
- moved Q3 77.1 mm to (124.4, 106.3)
- moved R26 77.0 mm to (127.4, 106.3), turned to -90 degrees
- moved C31 76.6 mm to (113.6, 106.0), turned to -90 degrees
- moved R23 75.7 mm to (120.6, 105.2)
- moved R27 75.5 mm to (117.1, 105.0)
- moved R43 74.5 mm to (120.7, 46.0)
- moved Q10 73.4 mm to (117.1, 46.9), turned to -90 degrees
- moved R22 73.4 mm to (120.6, 103.2)
- moved R21 73.3 mm to (113.6, 47.1), turned to -90 degrees
- moved Q2 73.0 mm to (124.4, 102.8)
- moved C36 72.9 mm to (127.5, 47.4), turned to -90 degrees
- moved C30 72.7 mm to (127.4, 102.6), turned to -90 degrees
- moved Q11 72.7 mm to (124.5, 47.6)
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Routing:
- net +5V: track 93.1 -> 275.6 mm, vias 0 -> 6
- net Net-(D14-K): track 0.00 -> 86.5 mm, vias 0 -> 2
- net Net-(D15-K): track 0.00 -> 61.5 mm, vias 0 -> 2
- net +3V3: track 52.6 -> 109.1 mm
- net Net-(D16-K): track 0.00 -> 43.5 mm, vias 0 -> 2
- net /leds_indication/led_indication_0/INDICATION: track 0.00 -> 36.4 mm, vias 0 -> 2
- net Net-(D17-K): track 0.00 -> 28.0 mm
- net /leds_indication/led_indication_3/INDICATION: track 0.00 -> 25.5 mm, vias 0 -> 2
- net /PWREN: track 9.15 -> 32.6 mm, vias 0 -> 2
- net Net-(D12-K): track 0.00 -> 22.6 mm
- net /eeprom/EECLK: track 17.4 -> 38.1 mm, vias 0 -> 2
- net /leds_indication/led_indication_1/INDICATION: track 0.00 -> 19.7 mm, vias 0 -> 2
- net /LIN 1/LIN: track 0.00 -> 19.1 mm
- net /eeprom/EEDATA: track 7.86 -> 26.2 mm, vias 0 -> 2
- net +1V8: track 22.9 -> 39.8 mm, vias 0 -> 4
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- added copper zone on B.Cu, net GND
- added copper zone on F.Cu, net GND

Commit message: all connected
Parts:
- moved R16 0.82 mm to (127.4, 61.6), turned to 180 degrees
Routing:
- net GND: track 18.2 -> 129.7 mm, vias 62 -> 86
- net /VBAT2: track 14.4 -> 20.9 mm
- net /VBAT3: track 14.7 -> 21.1 mm
- net Net-(D13-K): track 22.3 -> 25.6 mm
- net Net-(Q6-C): track 4.21 -> 6.59 mm
- net Net-(D8-K): track 1.84 -> 3.26 mm
- net /LIN0_RXD: track 53.8 -> 53.0 mm

Commit message: labels
Routing:
- net GND: track 129.7 -> 127.7 mm, vias 86 -> 117
- net /eeprom/EECLK: track 38.1 -> 36.6 mm
- net /VBAT2: track 20.9 -> 20.4 mm
- net (no net): vias 1 -> 0
Other:
- board text added: "VBAT"
- board text removed: "+"
