File: ftdi_quad_lin.kicad_sch (KiCad schematic)
At the start: 55 parts, among them J1 USB_C_Receptacle_USB2.0_16P, J6 Conn_01x10, J8 Barrel_Jack_MountingPin, U1 FT4232H, U3 AP2112K-3.3, U4 93CxxB, U8 74HC595, Y1 12Mhz

Commit message: Using bus
Parts:
- removed C25, C26: 100nF, Capacitor_SMD:C_0805_2012Metric, symbol Device:C
- removed D9: ~, ftdi_quad_lin:1296.3004, symbol ftdi_quad_lin:led_array_4
- removed R17, R19, R20, R21: 330R, Resistor_SMD:R_0805_2012Metric, symbol Device:R
- removed R18, R2, R6, R7: 10k, Resistor_SMD:R_0805_2012Metric, symbol Device:R
- removed R8: 2.2k, Resistor_SMD:R_0805_2012Metric, symbol Device:R
- removed U4: 93CxxB, Package_SO:SOIC-8_3.9x4.9mm_P1.27mm, symbol Memory_EEPROM:93CxxB
- removed U8: 74HC595, Package_SO:SOIC-16_3.9x9.9mm_P1.27mm, symbol 74xx:74HC595
Connections:
- no-connect marks 34 -> 29
Other:
- added sheet eeprom (eeprom.kicad_sch)
- added sheet leds_indication (leds_indication.kicad_sch)

Commit message: progress
Parts:
- removed D10: ~, ftdi_quad_lin:1296.3004, symbol ftdi_quad_lin:led_array_4
- removed R22, R23, R24, R25: 2.4k, Resistor_SMD:R_0805_2012Metric, symbol Device:R
Other:
- sheet leds_indication ports: added VBAT[0..3]; removed none

Commit message: Added manfs
Parts:
- FB2, FB3: manf# (none) -> BLM18AG601SN1D
- U1: manf# (none) -> FT4232HL-REEL
Changed lines of the file:
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@@
+			)
+		)
+		(property "manf#" "BLM18AG601SN1D"
+			(at 78.74 21.59 90)
+			(effects
+				(font
+					(size 1.27 1.27)
+				)
+				(hide yes)
 			)
 		)
@@
 		(property "Description" "Ferrite bead, small symbol"
 			(at 78.74 31.75 0)
+			(effects
+				(font
+					(size 1.27 1.27)
+				)
+				(hide yes)
+			)
+		)
+		(property "manf#" "BLM18AG601SN1D"
+			(at 78.74 31.75 90)
 			(effects
 				(font
@@
 			(at 151.13 109.22 0)
 			(effects
+				(font
+					(size 1.27 1.27)
+				)
+				(hide yes)
+			)
+		)
+		(property "manf#" "FT4232HL-REEL"
+			(at 151.13 109.22 0)
+			(effects

Commit message: pulldown reset
Parts:
- added R46: 100k, Resistor_SMD:R_0805_2012Metric, symbol Device:R
Connections:
- net GND: now also R46.2
- net at JP9.1 (A), R1.1, U1.14 (~{RESET}): now also R46.1
Other:
- moved on the sheet: R1, R3
Changed lines of the file:
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@@
 	)
 	(junction
+		(at 110.49 99.06)
+		(diameter 0)
+		(color 0 0 0 0)
+	)
+	(junction
 		(at 151.13 163.83)
 		(diameter 0)
@@
 	(wire
 		(pts
-			(xy 102.87 93.98) (xy 102.87 99.06)
+			(xy 90.17 93.98) (xy 90.17 99.06)
 		)
 		(stroke
@@
 	(wire
 		(pts
-			(xy 120.65 93.98) (xy 102.87 93.98)
+			(xy 120.65 93.98) (xy 90.17 93.98)
 		)
 		(stroke
@@
 	(wire
 		(pts
-			(xy 118.11 99.06) (xy 119.38 99.06)
+			(xy 107.95 99.06) (xy 110.49 99.06)
 		)
 		(stroke
@@
 	(wire
 		(pts
+			(xy 110.49 111.76) (xy 110.49 109.22)
+		)
+		(stroke
+			(width 0)
+			(type default)
+		)
+	)
+	(wire
+		(pts
 			(xy 196.85 157.48) (xy 224.79 157.48)
 		)
@@
 	(wire
 		(pts
-			(xy 102.87 106.68) (xy 102.87 110.49)
+			(xy 90.17 106.68) (xy 90.17 110.49)
 		)
 		(stroke
@@
 	(wire
 		(pts
-			(xy 107.95 97.79) (xy 107.95 99.06)
+			(xy 97.79 97.79) (xy 97.79 99.06)
 		)
 		(stroke
@@
 	(wire
 		(pts
+			(xy 110.49 99.06) (xy 110.49 101.6)
+		)
+		(stroke
+			(width 0)
+			(type default)
+		)
+	)
+	(wire
+		(pts
 			(xy 68.58 21.59) (xy 76.2 21.59)
 		)
@@
 	(wire
 		(pts
-			(xy 107.95 99.06) (xy 110.49 99.06)
+			(xy 97.79 99.06) (xy 100.33 99.06)
 		)
 		(stroke
@@
 	(wire
 		(pts
+			(xy 110.49 99.06) (xy 119.38 99.06)
+		)
+		(stroke
+			(width 0)
+			(type default)
+		)
+	)
+	(wire
+		(pts
 			(xy 113.03 66.04) (xy 113.03 49.53)
 		)
@@
 	(symbol
 		(lib_id "power:GND")
-		(at 102.87 110.49 0)
+		(at 90.17 110.49 0)
 		(unit 1)
 		(exclude_from_sim no)
@@
 		(fields_autoplaced yes)
 		(property "Reference" "#PWR019"
-			(at 102.87 116.84 0)
+			(at 90.17 116.84 0)
 			(effects
 				(font
@@
 		)
 		(property "Value" "GND"
-			(at 102.87 115.57 0)
+			(at 90.17 115.57 0)
 			(effects
 				(font
@@
 		)
 		(property "Footprint" ""
-			(at 102.87 110.49 0)
+			(at 90.17 110.49 0)
 			(effects
 				(font
@@
 		)
 		(property "Datasheet" ""
-			(at 102.87 110.49 0)
+			(at 90.17 110.49 0)
 			(effects
 				(font
@@
 		)
 		(property "Description" "Power symbol creates a global label with name \"GND\" , ground"
-			(at 102.87 110.49 0)
+			(at 90.17 110.49 0)
 			(effects
 				(font
@@
 	(symbol
 		(lib_id "power:GND")
+		(at 110.49 111.76 0)
+		(unit 1)
+		(exclude_from_sim no)
+		(in_bom yes)
+		(on_board yes)
+		(dnp no)
+		(fields_autoplaced yes)
+		(property "Reference" "#PWR090"
+			(at 110.49 118.11 0)
+			(effects
+				(font
+					(size 1.27 1.27)
+				)
+				(hide yes)
+			)
+		)
+		(property "Value" "GND"
+			(at 110.49 116.84 0)
+			(effects
+				(font
+					(size 1.27 1.27)
+				)
+				(hide yes)
+			)
+		)
+		(property "Footprint" ""
+			(at 110.49 111.76 0)
+			(effects
+				(font
+					(size 1.27 1.27)
+				)
+				(hide yes)
+			)
+		)
+		(property "Datasheet" ""
+			(at 110.49 111.76 0)
+			(effects
+				(font
+					(size 1.27 1.27)
+				)
+				(hide yes)
+			)
+		)
+		(property "Description" "Power symbol creates a global label with name \"GND\" , ground"
+			(at 110.49 111.76 0)
+			(effects
+				(font
+					(size 1.27 1.27)
+				)
+				(hide yes)
+			)
+		)
+		(pin "1"
+		)
+		(instances
+			(project "ftdi_quad_lin"
+				(path "/e6cf11d6-0152-4d84-a82a-9e2d93966152"
+					(reference "#PWR090")
+					(unit 1)
+				)
+			)
+		)
+	)
+	(symbol
+		(lib_id "power:GND")
 		(at 48.26 40.64 0)
 		(unit 1)
@@
 	(symbol
 		(lib_id "power:+3V3")
-		(at 107.95 97.79 0)
+		(at 97.79 97.79 0)
 		(unit 1)
 		(exclude_from_sim no)
@@
 		(dnp no)
 		(property "Reference" "#PWR020"
-			(at 107.95 101.6 0)
+			(at 97.79 101.6 0)
 			(effects
 				(font
@@
 		)
 		(property "Value" "+3V3"
-			(at 111.252 96.012 0)
+			(at 101.092 96.012 0)
 			(effects
 				(font
@@
 		)
 		(property "Footprint" ""
-			(at 107.95 97.79 0)
+			(at 97.79 97.79 0)
 			(effects
 				(font
@@
 		)
 		(property "Datasheet" ""
-			(at 107.95 97.79 0)
+			(at 97.79 97.79 0)
 			(effects
 				(font
@@
 		)
 		(property "Description" "Power symbol creates a global label with name \"+3V3\""
-			(at 107.95 97.79 0)
+			(at 97.79 97.79 0)
 			(effects
 				(font
@@
 	(symbol
 		(lib_id "Device:R")
-		(at 114.3 99.06 270)
+		(at 104.14 99.06 270)
 		(unit 1)
 		(exclude_from_sim no)
@@
 		(dnp no)
 		(property "Reference" "R1"
-			(at 114.3 99.06 90)
+			(at 104.14 99.06 90)
 			(effects
 				(font
@@
 		)
 		(property "Value" "1k"
-			(at 114.3 101.346 90)
+			(at 104.14 101.346 90)
 			(effects
 				(font
@@
 		)
 		(property "Footprint" "Resistor_SMD:R_0805_2012Metric"
-			(at 114.3 97.282 90)
+			(at 104.14 97.282 90)
 			(effects
 				(font
@@
 		)
 		(property "Datasheet" "~"
-			(at 114.3 99.06 0)
+			(at 104.14 99.06 0)
 			(effects
 				(font
@@
 		)
 		(property "Description" "Resistor"
-			(at 114.3 99.06 0)
+			(at 104.14 99.06 0)
 			(effects
 				(font
@@
 	(symbol
 		(lib_id "Device:R")
-		(at 102.87 102.87 180)
+		(at 110.49 105.41 0)
+		(unit 1)
+		(exclude_from_sim no)
+		(in_bom yes)
+		(on_board yes)
+		(dnp no)
+		(property "Reference" "R46"
+			(at 110.49 105.41 90)
+			(effects
+				(font
+					(size 1.27 1.27)
+				)
+			)
+		)
+		(property "Value" "100k"
+			(at 112.776 105.41 90)
+			(effects
+				(font
+					(size 1.27 1.27)
+				)
+			)
+		)
+		(property "Footprint" "Resistor_SMD:R_0805_2012Metric"
+			(at 108.712 105.41 90)
+			(effects
+				(font
+					(size 1.27 1.27)
+				)
+				(hide yes)
+			)
+		)
+		(property "Datasheet" "~"
+			(at 110.49 105.41 0)
+			(effects
+				(font
+					(size 1.27 1.27)
+				)
+				(hide yes)
+			)
+		)
+		(property "Description" "Resistor"
+			(at 110.49 105.41 0)
+			(effects
+				(font
+					(size 1.27 1.27)
+				)
+				(hide yes)
+			)
+		)
+		(pin "2"
+		)
+		(pin "1"
+		)
+		(instances
+			(project "ftdi_quad_lin"
+				(path "/e6cf11d6-0152-4d84-a82a-9e2d93966152"
+					(reference "R46")
+					(unit 1)
+				)
+			)
+		)
+	)
+	(symbol
+		(lib_id "Device:R")
+		(at 90.17 102.87 180)
 		(unit 1)
 		(exclude_from_sim no)
@@
 		(dnp no)
 		(property "Reference" "R3"
-			(at 102.87 102.87 90)
+			(at 90.17 102.87 90)
 			(effects
 				(font
@@
 		)
 		(property "Value" "12k"
-			(at 100.584 102.87 90)
+			(at 87.884 102.87 90)
 			(effects
 				(font
@@
 		)
 		(property "Footprint" "Resistor_SMD:R_0805_2012Metric"
-			(at 104.648 102.87 90)
+			(at 91.948 102.87 90)
 			(effects
 				(font
@@
 		)
 		(property "Datasheet" "~"
-			(at 102.87 102.87 0)
+			(at 90.17 102.87 0)
 			(effects
 				(font
@@
 		)
 		(property "Description" "Resistor"
-			(at 102.87 102.87 0)
+			(at 90.17 102.87 0)
 			(effects
 				(font
