File: lin.kicad_sch (KiCad schematic)
At the start: 10 parts, among them J3 Screw_Terminal_01x03, U5 TJA1029T

Commit message: routed
Parts:
- U5: symbol Interface_CAN_LIN:TJA1029TK -> Interface_CAN_LIN:TJA1029T
Connections:
- net GND: no longer U5.9 (GND)
- net VBAT: now reaches D3.2 (A), J3.1 (Pin_1), JP5.2 (B)
Changed lines of the file:
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@@
-	)
-	(junction
-		(at 120.65 111.76)
-		(diameter 0)
-		(color 0 0 0 0)
 	)
 	(junction
@@
 	)
 	(junction
+		(at 176.53 91.44)
+		(diameter 0)
+		(color 0 0 0 0)
+	)
+	(junction
 		(at 176.53 93.98)
 		(diameter 0)
@@
 	(wire
 		(pts
-			(xy 120.65 111.76) (xy 120.65 109.22)
+			(xy 120.65 109.22) (xy 120.65 114.3)
 		)
 		(stroke
@@
 	(wire
 		(pts
-			(xy 123.19 109.22) (xy 123.19 111.76)
-		)
-		(stroke
-			(width 0)
-			(type default)
-		)
-	)
-	(wire
-		(pts
 			(xy 133.35 101.6) (xy 160.02 101.6)
 		)
@@
 	(wire
 		(pts
-			(xy 176.53 90.17) (xy 176.53 93.98)
+			(xy 176.53 90.17) (xy 176.53 91.44)
 		)
 		(stroke
@@
 	(wire
 		(pts
-			(xy 120.65 114.3) (xy 120.65 111.76)
-		)
-		(stroke
-			(width 0)
-			(type default)
-		)
-	)
-	(wire
-		(pts
 			(xy 200.66 93.98) (xy 195.58 93.98)
 		)
@@
 	(wire
 		(pts
+			(xy 180.34 91.44) (xy 176.53 91.44)
+		)
+		(stroke
+			(width 0)
+			(type default)
+		)
+	)
+	(wire
+		(pts
 			(xy 152.4 87.63) (xy 160.02 87.63)
 		)
@@
 	(wire
 		(pts
+			(xy 176.53 91.44) (xy 176.53 93.98)
+		)
+		(stroke
+			(width 0)
+			(type default)
+		)
+	)
+	(wire
+		(pts
 			(xy 176.53 93.98) (xy 185.42 93.98)
 		)
@@
 		(pts
 			(xy 120.65 76.2) (xy 166.37 76.2)
-		)
-		(stroke
-			(width 0)
-			(type default)
-		)
-	)
-	(wire
-		(pts
-			(xy 123.19 111.76) (xy 120.65 111.76)
 		)
 		(stroke
@@
 			)
 			(justify right bottom)
+		)
+	)
+	(hierarchical_label "VBAT"
+		(shape input)
+		(at 180.34 91.44 0)
+		(fields_autoplaced yes)
+		(effects
+			(font
+				(size 1.27 1.27)
+			)
+			(justify left)
 		)
 	)
@@
 	)
 	(symbol
-		(lib_id "Interface_CAN_LIN:TJA1029TK")
+		(lib_id "Interface_CAN_LIN:TJA1029T")
 		(at 120.65 99.06 0)
 		(unit 1)
@@
 			)
 		)
-		(property "Description" "LIN 2.2A/SAE J2602 transceiver with TXD dominant timeout, DFN-8"
+		(property "Description" "LIN 2.2A/SAE J2602 transceiver with TXD dominant timeout, SOIC-8"
 			(at 120.65 99.06 0)
 			(effects
@@
 		(pin "8"
 		)
-		(pin "9"
-		)
 		(pin "1"

Commit message: Using bus
Parts:
- renumbered JP5 to JP6
Changed lines of the file:
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@@
 	(label "LIN"
 		(at 181.61 101.6 180)
-		(fields_autoplaced yes)
 		(effects
 			(font
@@
 		(shape input)
 		(at 180.34 91.44 0)
-		(fields_autoplaced yes)
 		(effects
 			(font
@@
 		(shape input)
 		(at 88.9 93.98 180)
-		(fields_autoplaced yes)
 		(effects
 			(font
@@
 		(shape input)
 		(at 88.9 96.52 180)
-		(fields_autoplaced yes)
 		(effects
 			(font
@@
 		(on_board yes)
 		(dnp no)
-		(property "Reference" "JP5"
+		(property "Reference" "JP6"
 			(at 190.5 91.948 0)
 			(effects
@@
 		(dnp no)
 		(fields_autoplaced yes)
-		(property "Reference" "#PWR069"
+		(property "Reference" "#PWR083"
 			(at 200.66 95.25 0)
 			(effects

Commit message: progress
Connections:
- net VBAT: now also C18.1, D3.1 (K), JP2.1 (A), U5.7 (VBAT); no longer D3.2 (A), J3.1 (Pin_1), JP6.2 (B)
- new net: D3.2 (A), J3.1 (Pin_1), JP6.2 (B)

Commit message: new connectors
Parts:
- J3: footprint TerminalBlock:TerminalBlock_Xinya_XY308-2.54-3P_1x03_P2.54mm_Horizontal -> ftdi_quad_lin:lin_connector
Changed lines of the file:
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@@
 			)
 		)
-		(property "Footprint" "TerminalBlock:TerminalBlock_Xinya_XY308-2.54-3P_1x03_P2.54mm_Horizontal"
+		(property "Footprint" "ftdi_quad_lin:lin_connector"
 			(at 186.69 101.6 0)
 			(effects

Commit message: Added manfs
Parts:
- U5: manf# (none) -> TJA1029T,118
Changed lines of the file:
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@@
 		(on_board yes)
 		(dnp no)
-		(fields_autoplaced yes)
 		(property "Reference" "D3"
-			(at 179.07 85.7249 90)
+			(at 178.308 86.36 90)
 			(effects
 				(font
@@
 			)
 		)
+		(property "manf#" "TJA1029T,118"
+			(at 120.65 99.06 0)
+			(effects
+				(font
+					(size 1.27 1.27)
+				)
+				(hide yes)
+			)
+		)
 		(pin "8"
 		)
@@
 		(on_board yes)
 		(dnp no)
-		(fields_autoplaced yes)
 		(property "Reference" "D4"
-			(at 148.59 82.55 0)
-			(effects
-				(font
+			(at 148.844 84.836 0)
+			(effects
+				(font

Commit message: added ESD protection to lin
Parts:
- added D19: ESD1LIN24, Diode_SMD:D_SOD-323_HandSoldering, symbol Diode:SD05_SOD323
Connections:
- net GND: now also D19.1 (A1)
- net LIN: now also D19.2 (A2)
Changed lines of the file:
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@@
 		(color 0 0 0 0)
 	)
-	(wire
-		(pts
-			(xy 160.02 101.6) (xy 181.61 101.6)
+	(junction
+		(at 170.18 101.6)
+		(diameter 0)
+		(color 0 0 0 0)
+	)
+	(wire
+		(pts
+			(xy 160.02 101.6) (xy 170.18 101.6)
 		)
 		(stroke
@@
 	(wire
 		(pts
+			(xy 170.18 101.6) (xy 181.61 101.6)
+		)
+		(stroke
+			(width 0)
+			(type default)
+		)
+	)
+	(wire
+		(pts
 			(xy 140.97 87.63) (xy 144.78 87.63)
 		)
@@
 	(wire
 		(pts
-			(xy 181.61 104.14) (xy 177.8 104.14)
+			(xy 181.61 104.14) (xy 180.34 104.14)
 		)
 		(stroke
@@
 		(pts
 			(xy 176.53 90.17) (xy 176.53 93.98)
+		)
+		(stroke
+			(width 0)
+			(type default)
+		)
+	)
+	(wire
+		(pts
+			(xy 170.18 102.87) (xy 170.18 101.6)
 		)
 		(stroke
@@
 	(symbol
 		(lib_id "power:GND")
-		(at 177.8 104.14 0)
+		(at 180.34 104.14 0)
 		(unit 1)
 		(exclude_from_sim no)
@@
 		(fields_autoplaced yes)
 		(property "Reference" "#PWR059"
-			(at 177.8 110.49 0)
+			(at 180.34 110.49 0)
 			(effects
 				(font
@@
 		)
 		(property "Value" "GND"
-			(at 177.8 109.22 0)
+			(at 180.34 109.22 0)
 			(effects
 				(font
@@
 		)
 		(property "Footprint" ""
-			(at 177.8 104.14 0)
+			(at 180.34 104.14 0)
 			(effects
 				(font
@@
 		)
 		(property "Datasheet" ""
-			(at 177.8 104.14 0)
+			(at 180.34 104.14 0)
 			(effects
 				(font
@@
 		)
 		(property "Description" "Power symbol creates a global label with name \"GND\" , ground"
-			(at 177.8 104.14 0)
+			(at 180.34 104.14 0)
 			(effects
 				(font
@@
 	)
 	(symbol
+		(lib_id "power:GND")
+		(at 170.18 110.49 0)
+		(unit 1)
+		(exclude_from_sim no)
+		(in_bom yes)
+		(on_board yes)
+		(dnp no)
+		(fields_autoplaced yes)
+		(property "Reference" "#PWR0120"
+			(at 170.18 116.84 0)
+			(effects
+				(font
+					(size 1.27 1.27)
+				)
+				(hide yes)
+			)
+		)
+		(property "Value" "GND"
+			(at 170.18 115.57 0)
+			(effects
+				(font
+					(size 1.27 1.27)
+				)
+				(hide yes)
+			)
+		)
+		(property "Footprint" ""
+			(at 170.18 110.49 0)
+			(effects
+				(font
+					(size 1.27 1.27)
+				)
+				(hide yes)
+			)
+		)
+		(property "Datasheet" ""
+			(at 170.18 110.49 0)
+			(effects
+				(font
+					(size 1.27 1.27)
+				)
+				(hide yes)
+			)
+		)
+		(property "Description" "Power symbol creates a global label with name \"GND\" , ground"
+			(at 170.18 110.49 0)
+			(effects
+				(font
+					(size 1.27 1.27)
+				)
+				(hide yes)
+			)
+		)
+		(pin "1"
+		)
+		(instances
+			(project "ftdi_quad_lin"
+				(path "/e6cf11d6-0152-4d84-a82a-9e2d93966152/31c6b4ae-10a2-4f10-a591-5579630fa60e"
+					(reference "#PWR0121")
+					(unit 1)
+				)
+				(path "/e6cf11d6-0152-4d84-a82a-9e2d93966152/7747294f-2018-4c44-a2cb-fbe0ffa31304"
+					(reference "#PWR0123")
+					(unit 1)
+				)
+				(path "/e6cf11d6-0152-4d84-a82a-9e2d93966152/a2f7cee2-a97f-4885-9036-e6c309dcb8d0"
+					(reference "#PWR0122")
+					(unit 1)
+				)
+				(path "/e6cf11d6-0152-4d84-a82a-9e2d93966152/ce397451-b7a0-48ce-ab00-72bbf812467b"
+					(reference "#PWR0120")
+					(unit 1)
+				)
+			)
+		)
+	)
+	(symbol
 		(lib_id "Device:C")
 		(at 160.02 106.68 0)
@@
 					(unit 1)
 				)
+			)
+		)
+	)
+	(symbol
+		(lib_id "Diode:SD05_SOD323")
+		(at 170.18 106.68 90)
+		(unit 1)
+		(exclude_from_sim no)
+		(in_bom yes)
+		(on_board yes)
+		(dnp no)
+		(fields_autoplaced yes)
+		(property "Reference" "D19"
+			(at 172.72 105.4099 90)
+			(effects
+				(font
+					(size 1.27 1.27)
+				)
+				(justify right)
+			)
+		)
+		(property "Value" "ESD1LIN24"
+			(at 172.72 107.9499 90)
+			(effects
+				(font
+					(size 1.27 1.27)
+				)
+				(justify right)
+			)
+		)
+		(property "Footprint" "Diode_SMD:D_SOD-323_HandSoldering"
+			(at 175.26 106.68 0)
+			(effects
+				(font
+					(size 1.27 1.27)
+				)
+				(hide yes)
+			)
+		)
+		(property "Datasheet" "https://www.littelfuse.com/~/media/electronics/datasheets/tvs_diode_arrays/littelfuse_tvs_diode_array_sd_c_datasheet.pdf.pdf"
+			(at 170.18 106.68 0)
+			(effects
+				(font
+					(size 1.27 1.27)
+				)
+				(hide yes)
+			)
+		)
+		(property "Description" "5V, 450W Discrete Bidirectional TVS Diode, SOD-323"
+			(at 170.18 106.68 0)
+			(effects
+				(font
+					(size 1.27 1.27)
+				)
+				(hide yes)
+			)
+		)
+		(pin "2"
+		)
+		(pin "1"
+		)
+		(instances
+			(project ""
+				(path "/e6cf11d6-0152-4d84-a82a-9e2d93966152/31c6b4ae-10a2-4f10-a591-5579630fa60e"
+					(reference "D18")
+					(unit 1)
+				)
+				(path "/e6cf11d6-0152-4d84-a82a-9e2d93966152/7747294f-2018-4c44-a2cb-fbe0ffa31304"
+					(reference "D20")
+					(unit 1)
+				)
+				(path "/e6cf11d6-0152-4d84-a82a-9e2d93966152/a2f7cee2-a97f-4885-9036-e6c309dcb8d0"
+					(reference "D19")
+					(unit 1)
+				)
+				(path "/e6cf11d6-0152-4d84-a82a-9e2d93966152/ce397451-b7a0-48ce-ab00-72bbf812467b"
+					(reference "D9")
+					(unit 1)
+				)
