File: led_indication.kicad_sch (KiCad schematic)
At the start: 12 parts, among them Q7 MMBT2222A, Q8 MMBT2222A, Q9 MMBT2222A

Commit message: Added manfs
Parts:
- Q7, Q8, Q9: manf# (none) -> MMBT2222A
Changed lines of the file:
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@@
+			)
+		)
+		(property "manf#" "MMBT2222A"
+			(at 179.07 85.09 0)
+			(effects
+				(font
+					(size 1.27 1.27)
+				)
+				(hide yes)
 			)
 		)
@@
 			)
 		)
+		(property "manf#" "MMBT2222A"
+			(at 144.78 85.09 0)
+			(effects
+				(font
+					(size 1.27 1.27)
+				)
+				(hide yes)
+			)
+		)
 		(pin "2"
 		)
@@
 			(at 121.92 73.66 0)
 			(effects
+				(font
+					(size 1.27 1.27)
+				)
+				(hide yes)
+			)
+		)
+		(property "manf#" "MMBT2222A"
+			(at 121.92 73.66 0)
+			(effects

Commit message: 1M ohm
Parts:
- R35: value 330k -> 1M
Changed lines of the file:
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@@
 			)
 		)
-		(property "Value" "330k"
+		(property "Value" "1M"
 			(at 158.496 58.42 90)
 			(effects
