File: hw/ftdi_quad_lin.kicad_pcb (KiCad board)
At the start: 2 copper layers, 55 x 80 mm, 157 parts, among them J1 USB_C_Receptacle_USB2.0_16P, J2 Screw_Terminal_01x03, J3 Screw_Terminal_01x03, J4 Screw_Terminal_01x03, J5 Screw_Terminal_01x03, J6 Conn_01x10, J7 Conn_01x05, J8 Barrel_Jack_MountingPin, Q1 MMBT2222A, Q10 MMBT2222A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

Commit message: fixes
Routing:
- net +5V: track 301.4 -> 299.3 mm
- net GND: track 123.3 -> 124.6 mm, vias 115 -> 117
- net Net-(D15-K): track 59.2 -> 59.8 mm

Commit message: fixes
Routing:
- net /LIN1_TXD: track 54.5 -> 55.3 mm
Changed lines of the file:
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@@
-	)
-	(segment
-		(start 102.62241 109.77759)
-		(end 102.62241 91.6)
-		(width 0.2)
-		(layer "F.Cu")
-		(net 83)
 	)
 	(segment
@@
 	)
 	(segment
+		(start 102.62241 89.8)
+		(end 102.62241 89.295076)
+		(width 0.2)
+		(layer "F.Cu")
+		(net 83)
+	)
+	(segment
+		(start 102.62241 109.77759)
+		(end 102.62241 89.8)
+		(width 0.2)
+		(layer "F.Cu")
+		(net 83)
+	)
+	(segment
 		(start 100.909744 87.58241)
 		(end 102.62241 89.295076)
@@
 		(start 117.7 97.08625)
 		(end 116.28625 97.08625)
-		(width 0.2)
-		(layer "F.Cu")
-		(net 83)
-	)
-	(segment
-		(start 102.62241 91.6)
-		(end 102.62241 89.295076)
 		(width 0.2)
 		(layer "F.Cu")
@@
 	)
 	(via
-		(at 102.62241 91.6)
+		(at 102.62241 89.8)
 		(size 0.6)
 		(drill 0.3)
@@
 	)
 	(segment
-		(start 116.2 97)
-		(end 108.02241 97)
+		(start 109 92.8)
+		(end 113.2 97)
 		(width 0.2)
 		(layer "B.Cu")
@@
 	)
 	(segment
-		(start 108.02241 97)
-		(end 102.62241 91.6)
+		(start 105.62241 92.8)
+		(end 102.62241 89.8)
+		(width 0.2)
+		(layer "B.Cu")
+		(net 83)
+	)
+	(segment
+		(start 109 92.8)
+		(end 105.62241 92.8)
+		(width 0.2)
+		(layer "B.Cu")
+		(net 83)
+	)
+	(segment
+		(start 113.2 97)
+		(end 116.2 97)
 		(width 0.2)
 		(layer "B.Cu")
@@
 	)
 	(segment
-		(start 110.90061 68.2)
-		(end 108.10061 71)
+		(start 109 71)
+		(end 111.8 68.2)
 		(width 0.2)
 		(layer "B.Cu")
@@
 	)
 	(segment
-		(start 111.8 68.2)
-		(end 110.90061 68.2)
-		(width 0.2)
-		(layer "B.Cu")
-		(net 101)
-	)
-	(segment
-		(start 108.10061 71)
-		(end 100.8 71)
+		(start 100.8 71)
+		(end 109 71)
 		(width 0.2)
 		(layer "B.Cu")
@@
 	)
 	(segment
-		(start 119.259222 60.626667)
-		(end 100.676667 60.626667)
+		(start 100.8 60.8)
+		(end 119.432556 60.8)
+		(width 1)
+		(layer "B.Cu")
+		(net 130)
+	)
+	(segment
+		(start 100.676667 60.626667)
+		(end 100.676667 60.676667)
 		(width 1)
 		(layer "B.Cu")
@@
 	)
 	(segment
+		(start 119.432556 60.8)
+		(end 119.716278 61.083722)
+		(width 1)
+		(layer "B.Cu")
+		(net 130)
+	)
+	(segment
+		(start 129.6 70.967445)
+		(end 119.716278 61.083722)
+		(width 1)
+		(layer "B.Cu")
+		(net 130)
+	)
+	(segment
 		(start 130 98.43083)
 		(end 129.6 98.03083)
@@
 	)
 	(segment
-		(start 129.6 70.967445)
-		(end 119.259222 60.626667)
+		(start 100.676667 60.676667)
+		(end 100.8 60.8)
 		(width 1)
 		(layer "B.Cu")
