File: hw/ftdi_quad_lin.kicad_pcb (KiCad board)
At the start: 2 copper layers, 55 x 80 mm, 157 parts, among them J1 USB_C_Receptacle_USB2.0_16P, J2 Screw_Terminal_01x03, J3 Screw_Terminal_01x03, J4 Screw_Terminal_01x03, J5 Screw_Terminal_01x03, J6 Conn_01x10, J7 Conn_01x05, J8 Barrel_Jack_MountingPin, Q1 MMBT2222A, Q10 MMBT2222A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

Commit message: hw: led RC changed 220n->100n
Parts:
- C30, C32, C34, C36: value 220n -> 100n
