File: hw/ftdi_quad_lin.kicad_sch (KiCad schematic)
At the start: 37 parts, among them J1 USB_C_Receptacle_USB2.0_16P, J6 Conn_01x10, J8 Barrel_Jack_MountingPin, U1 FT4232H, U3 AP2112K-3.3, Y1 12Mhz

Commit message: hw: manf for jack
Parts:
- J8: manf# (none) -> PJ-063AH
Changed lines of the file:
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@@
+			)
+		)
+		(property "manf#" "PJ-063AH"
+			(at 115.57 181.61 0)
+			(effects
+				(font
+					(size 1.27 1.27)
+				)
+				(hide yes)
 			)
 		)

Commit message: hw: manf for USB
Parts:
- J1: manf# (none) -> USB4105-GF-A-120
Changed lines of the file:
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@@
+			)
+		)
+		(property "manf#" "USB4105-GF-A-120"
+			(at 50.8 86.36 0)
+			(effects
+				(font
+					(size 1.27 1.27)
+				)
+				(hide yes)
 			)
 		)
