File: hw/led_indication.kicad_sch (KiCad schematic)
At the start: 12 parts, among them Q7 MMBT2222A, Q8 MMBT2222A, Q9 MMBT2222A

Commit message: hw: led RC changed 220n->100n
Parts:
- C34: value 220n -> 100n
Changed lines of the file:
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@@
 			)
 		)
-		(property "Value" "220n"
+		(property "Value" "100n"
 			(at 149.86 68.58 90)
 			(effects
